Commit message: camera is added to robot

File: my_robot/urdf/my_robot.xacro (robot description, xacro)
@@ -113,3 +113,30 @@
     <dynamics damping="1.0" friction="1.0"/>
   </joint>
+  <link name='camera'>
+      <visual>
+        <origin xyz="0 0 0" rpy="0 0 0" />
+        <geometry>
+        <box size="0.05 0.05 0.05" />
+        </geometry>
+      </visual>
+      <collision>
+        <origin xyz="0 0 0" rpy="0 0 0" />
+        <geometry>
+        <box size="0.05 0.05 0.05" />
+        </geometry>
+      </collision>
+      <inertial>
+        <origin xyz="0 0 0"  rpy="0 0 0" />
+        <mass value="0.1" />
+        <inertia  ixx="0.000001" ixy="0" ixz="0"
+                  iyy="0.000001" iyz="0"
+                  izz="0.000001" />
+      </inertial>
+    </link>
+    <joint type="fixed" name="camera_joint">
+    <origin xyz="0.2 0 0" rpy="0 0 0"/>
+    <child link="camera"/>
+    <parent link="chassis"/>
+    <axis xyz="0 1 0" rpy="0 0 0"/>
+  </joint>
 </robot>

Commit message: Lidar sensor is added to robot

File: my_robot/urdf/my_robot.xacro (robot description, xacro)
@@ -140,3 +140,30 @@
     <axis xyz="0 1 0" rpy="0 0 0"/>
   </joint>
+  <link name='hokuyo'>
+      <visual>
+        <origin xyz="0 0 0" rpy="0 0 0" />
+        <geometry>
+        <mesh filename="package://my_robot/meshes/hokuyo.dae" />
+        </geometry>
+      </visual>
+      <collision>
+        <origin xyz="0 0 0" rpy="0 0 0" />
+        <geometry>
+        <box size="0.1 0.1 0.1" />
+        </geometry>
+      </collision>
+      <inertial>
+        <origin xyz="0 0 0"  rpy="0 0 0" />
+        <mass value="0.00001" />
+        <inertia  ixx="0.000001" ixy="0" ixz="0"
+                  iyy="0.000001" iyz="0"
+                  izz="0.000001" />
+      </inertial>
+    </link>
+    <joint type="fixed" name="hokuyo_joint">
+    <origin xyz="0.15 0 0.1" rpy="0 0 0"/>
+    <child link="hokuyo"/>
+    <parent link="chassis"/>
+    <axis xyz="0 1 0" rpy="0 0 0"/>
+  </joint>
 </robot>

Commit message: colors are added for robot

File: my_robot/urdf/my_robot.xacro (robot description, xacro)
@@ -7,4 +7,7 @@
     <child link="chassis" />
   </joint>
+  <gazebo reference="chassis">
+    <material>Gazebo/Orange</material>
+  </gazebo>
   <link name='chassis'>
     <pose>0 0 0.1 0 0 0</pose>
@@ -55,4 +58,7 @@
     </visual>
   </link>
+ <gazebo reference="right_wheel">
+    <material>Gazebo/Black</material>
+  </gazebo>
 <link name='right_wheel'>
       <visual>
@@ -84,4 +90,7 @@
     <dynamics damping="1.0" friction="1.0"/>
   </joint>
+  <gazebo reference="left_wheel">
+    <material>Gazebo/Black</material>
+  </gazebo>
   <link name='left_wheel'>
       <visual>
@@ -140,4 +149,7 @@
     <axis xyz="0 1 0" rpy="0 0 0"/>
   </joint>
+  <gazebo reference="camera">
+    <material>Gazebo/Black</material>
+  </gazebo>
   <link name='hokuyo'>
       <visual>

Commit message: suggested changes are done

File: my_robot/urdf/my_robot.xacro (robot description, xacro)
@@ -157,5 +157,5 @@
         <origin xyz="0 0 0" rpy="0 0 0" />
         <geometry>
-        <mesh filename="package://my_robot/meshes/hokuyo.dae" />
+        <mesh filename="$(find my_robot)/meshes/hokuyo.dae" />
         </geometry>
       </visual>

Commit message: camera optical link added

File: my_robot/urdf/my_robot.xacro (robot description, xacro)
@@ -150,4 +150,11 @@
     <axis xyz="0 1 0" rpy="0 0 0"/>
   </joint>
+  <joint name="camera_optical_joint" type="fixed">
+    <origin xyz="0 0 0" rpy="-1.5707 0 -1.5707"/>
+    <parent link="camera_link"/>
+    <child link="camera_link_optical"/>
+  </joint>
+  <link name="camera_link_optical">
+  </link>
   <gazebo reference="camera">
     <material>Gazebo/Black</material>
